Commit message: laser link was added in urdf model of robot

File: src/bumperbot_description/urdf/bumperbot.urdf.xacro (robot description, xacro)
@@ -175,3 +175,29 @@
     <axis xyz="0 0 0" />
   </joint>
+  <link name = "laser_link">
+    <inertial>
+        <origin xyz="-0.011945780406062 -0.000381929217680526 -0.0170649378129477" rpy="0 0 0" />
+        <mass value="0.073084435549317" />
+        <inertia ixx="1.96074931730795E-05" ixy="-3.62091076640009E-07" ixz="4.28230084046735E-07"
+                 iyy="2.40983835136327E-05" iyz="1.50180909250652E-08" izz="4.14184164228595E-05" />
+    </inertial>
+    <visual>
+      <origin xyx = "0 0 0" rpy = "0 0 0"/>
+      <geometry>
+        <mesh filename="package://bumperbot_description/meshes/laser_link.STL" />
+      </geometry>
+    </visual>
+     <collision>
+      <origin xyx = "0 0 0" rpy = "0 0 0"/>
+      <geometry>
+        <mesh filename="package://bumperbot_description/meshes/laser_link.STL" />
+      </geometry>
+    </collision>
+  </link>
+  <joint name="laser_joint" type="fixed">
+    <parent link="base_link" />
+    <child link="laser_link" />
+    <origin xyz="0.0 0.0 0.1208" rpy="0 0 3.14" />
+    <axis xyz="0 0 0" />
+  </joint>
 </robot>

Commit message: files and codes were added for map and localizaion

File: src/bumperbot_description/urdf/bumperbot.urdf.xacro (robot description, xacro)
@@ -23,4 +23,5 @@
         <mesh filename="package://bumperbot_description/meshes/base_link.STL" />
       </geometry>
+      <material name="black"/>
     </visual>
     <collision>
@@ -49,4 +50,5 @@
         <mesh filename="package://bumperbot_description/meshes/wheel_right_link.STL" />
       </geometry>
+      <material name="blue"/>
     </visual>
     <collision>
@@ -77,4 +79,5 @@
         <mesh filename="package://bumperbot_description/meshes/wheel_left_link.STL" />
       </geometry>
+      <material name="blue"/>
     </visual>
     <collision>
@@ -104,4 +107,5 @@
         <mesh filename="package://bumperbot_description/meshes/caster_front_link.STL" />
       </geometry>
+      <material name="silver"/>
     </visual>
     <collision>
@@ -131,4 +135,5 @@
         <mesh filename="package://bumperbot_description/meshes/caster_rear_link.STL" />
       </geometry>
+      <material name="silver"/>
     </visual>
     <collision>
@@ -158,7 +163,5 @@
         <mesh filename="package://bumperbot_description/meshes/imu_link.STL" />
       </geometry>
-      <material name="">
-        <color rgba="0.792156862745098 0.819607843137255 0.933333333333333 1" />
-      </material>
+      <material name="blue"/>
     </visual>
     <collision>
@@ -175,19 +178,21 @@
     <axis xyz="0 0 0" />
   </joint>
-  <link name = "laser_link">
-    <inertial>
-        <origin xyz="-0.011945780406062 -0.000381929217680526 -0.0170649378129477" rpy="0 0 0" />
-        <mass value="0.073084435549317" />
-        <inertia ixx="1.96074931730795E-05" ixy="-3.62091076640009E-07" ixz="4.28230084046735E-07"
-                 iyy="2.40983835136327E-05" iyz="1.50180909250652E-08" izz="4.14184164228595E-05" />
-    </inertial>
-    <visual>
-      <origin xyx = "0 0 0" rpy = "0 0 0"/>
+  <link name="laser_link">
+    <inertial>
+      <origin xyz="-0.011945780406062 -0.000381929217680526 -0.0170649378129477" rpy="0 0 0" />
+      <mass value="0.073084435549317" />
+      <inertia ixx="1.96074931730795E-05" ixy="-3.62091076640009E-07" ixz="4.28230084046735E-07"
+               iyy="2.40983835136327E-05" iyz="1.50180909250652E-08"
+               izz="4.14184164228595E-05" />
+    </inertial>
+    <visual>
+      <origin xyz="0 0 0" rpy="0 0 0" />
       <geometry>
         <mesh filename="package://bumperbot_description/meshes/laser_link.STL" />
       </geometry>
-    </visual>
-     <collision>
-      <origin xyx = "0 0 0" rpy = "0 0 0"/>
+      <material name="dark_grey"/>
+    </visual>
+    <collision>
+      <origin xyz="0 0 0" rpy="0 0 0" />
       <geometry>
         <mesh filename="package://bumperbot_description/meshes/laser_link.STL" />
@@ -196,8 +201,20 @@
   </link>
   <joint name="laser_joint" type="fixed">
+    <origin xyz="-0.0050526 -0.0023221 0.1208" rpy="0 0 3.14" />
     <parent link="base_link" />
     <child link="laser_link" />
-    <origin xyz="0.0 0.0 0.1208" rpy="0 0 3.14" />
-    <axis xyz="0 0 0" />
-  </joint>
+    <axis xyz="0 0 0" />
+  </joint>
+  <material name="blue">
+    <color rgba="0 0 1 1"/>
+  </material>
+  <material name="black">
+    <color rgba="0 0 0 1"/>
+  </material>
+  <material name="silver">
+    <color rgba="0.79 0.82 0.93 1"/>
+  </material>
+  <material name="dark_grey">
+    <color rgba="0.3 0.3 0.3 1"/>
+  </material>
 </robot>

File: src/bumperbot_description/urdf/bumperbot_ros2_control.xacro (robot description, xacro)
@@ -21,5 +21,5 @@
             <hardware>
                 <plugin>bumperbot_firmware/BumperbotInterface</plugin>
-                <param name="port">/dev/ttyACM0</param>
+                <param name="port">/dev/arduino</param>
             </hardware>
         </xacro:unless>
